File: PCB/nRF52840-FART/nRF52840-FART.kicad_sch (KiCad schematic)
At the start: 7 parts, among them U1 xiao-ble

Commit message: v0.2 of the PCB
Parts:
- BATT1, Probe1, Probe2: footprint TerminalBlock_TE-Connectivity:TerminalBlock_TE_282834-2_1x02_P2.54mm_Horizontal -> Connector_JST:JST_PH_S2B-PH-K_1x02_P2.00mm_Horizontal
Connections:
- net GND: no longer U1.13 (GND)
- now unconnected: U1.15 (A31_SWDIO), U1.16 (A30_SWCLK), U1.17 (RESET), U1.18 (GND)
- no-connect marks 14 -> 15
Changed lines of the file:
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@@
 	(paper "A4")
-	(junction
-		(at 151.13 71.12)
-		(diameter 0)
-		(color 0 0 0 0)
-	)
 	(junction
 		(at 64.77 111.76)
@@
 	)
 	(junction
-		(at 148.59 71.12)
-		(diameter 0)
-		(color 0 0 0 0)
-	)
-	(junction
 		(at 88.9 113.03)
 		(diameter 0)
@@
 	)
 	(no_connect
+		(at 171.45 81.28)
+	)
+	(no_connect
 		(at 128.27 93.98)
 	)
@@
 	(wire
 		(pts
-			(xy 151.13 71.12) (xy 153.67 71.12)
-		)
-		(stroke
-			(width 0)
-			(type default)
-		)
-	)
-	(wire
-		(pts
 			(xy 171.45 91.44) (xy 184.15 91.44)
 		)
@@
 	(wire
 		(pts
-			(xy 171.45 81.28) (xy 185.42 81.28)
-		)
-		(stroke
-			(width 0)
-			(type default)
-		)
-	)
-	(wire
-		(pts
 			(xy 66.04 77.47) (xy 68.58 77.47)
 		)
@@
 	(wire
 		(pts
-			(xy 148.59 71.12) (xy 151.13 71.12)
-		)
-		(stroke
-			(width 0)
-			(type default)
-		)
-	)
-	(wire
-		(pts
 			(xy 66.04 87.63) (xy 68.58 87.63)
 		)
@@
 		(pts
 			(xy 88.9 123.19) (xy 88.9 128.27)
-		)
-		(stroke
-			(width 0)
-			(type default)
-		)
-	)
-	(wire
-		(pts
-			(xy 146.05 71.12) (xy 148.59 71.12)
 		)
 		(stroke
@@
 		(fields_autoplaced yes)
 		(property "Reference" "BATT1"
-			(at 151.13 113.03 90)
+			(at 151.13 112.3949 90)
 			(effects
 				(font
@@
 		)
 		(property "Value" "Conn_01x02_Pin"
-			(at 151.13 115.57 90)
+			(at 151.13 114.9349 90)
 			(effects
 				(font
@@
 			)
 		)
-		(property "Footprint" "TerminalBlock_TE-Connectivity:TerminalBlock_TE_282834-2_1x02_P2.54mm_Horizontal"
+		(property "Footprint" "Connector_JST:JST_PH_S2B-PH-K_1x02_P2.00mm_Horizontal"
 			(at 149.86 113.03 0)
 			(effects
@@
 			)
 		)
-		(property "Footprint" "TerminalBlock_TE-Connectivity:TerminalBlock_TE_282834-2_1x02_P2.54mm_Horizontal"
+		(property "Footprint" "Connector_JST:JST_PH_S2B-PH-K_1x02_P2.00mm_Horizontal"
 			(at 67.31 104.14 0)
 			(effects
@@
 			)
 		)
-		(property "Footprint" "TerminalBlock_TE-Connectivity:TerminalBlock_TE_282834-2_1x02_P2.54mm_Horizontal"
+		(property "Footprint" "Connector_JST:JST_PH_S2B-PH-K_1x02_P2.00mm_Horizontal"
 			(at 91.44 104.14 0)
 			(effects
@@
 					(unit 1)
 				)
-			)
-		)
-	)
-	(symbol
-		(lib_id "power:GND")
-		(at 185.42 81.28 0)
-		(unit 1)
-		(exclude_from_sim no)
-		(in_bom yes)
-		(on_board yes)
-		(dnp no)
-		(fields_autoplaced yes)
-		(property "Reference" "#PWR010"
-			(at 185.42 87.63 0)
-			(effects
-				(font
-					(size 1.27 1.27)
-				)
-				(hide yes)
-			)
-		)
-		(property "Value" "GND"
-			(at 185.42 86.36 0)
-			(effects
-				(font
-					(size 1.27 1.27)
-				)
-			)
-		)
-		(property "Footprint" ""
-			(at 185.42 81.28 0)
-			(effects
-				(font
-					(size 1.27 1.27)
-				)
-				(hide yes)
-			)
-		)
-		(property "Datasheet" ""
-			(at 185.42 81.28 0)
-			(effects
-				(font
-					(size 1.27 1.27)
-				)
-				(hide yes)
-			)
-		)
-		(property "Description" ""
-			(at 185.42 81.28 0)
-			(effects
-				(font
-					(size 1.27 1.27)
-				)
-				(hide yes)
-			)
-		)
-		(pin "1"
-		)
-		(instances
-			(project "RadiatorBalancer"
-				(path "/9240e15d-484a-49b3-8f80-37d1a010783e"
-					(reference "#PWR010")
-					(unit 1)
-				)
